Commit message: updated collision meshes for tekken and increase damping of joints

File: source/fr3_tekken_adof/data/robots/tekken_adof/left_adof_qca/Left_adof_qca.urdf (robot description, URDF)
Before this commit: robot Left_adof_qca, 22 links, 21 joints
Links:
- link Index_Distal_Phalanx: geometry collision mesh filename=meshes/collmesh_DIP.STL; visual mesh filename=meshes/Index_Distal_Phalanx.STL
- link Index_MCP_Pitch: geometry collision mesh filename=meshes/Index_MCP_Pitch.STL; visual mesh filename=meshes/Index_MCP_Pitch.STL
- link Index_MCP_Yaw: geometry collision mesh filename=meshes/collmesh_PIP.STL; visual mesh filename=meshes/Index_MCP_Yaw.STL
- link Index_Middle_Phalanx: geometry collision mesh filename=meshes/collmesh_MIP.STL; visual mesh filename=meshes/Index_Middle_Phalanx.STL
- link Middle_Distal_Phalanx: geometry collision mesh filename=meshes/collmesh_DIP.STL; visual mesh filename=meshes/Middle_Distal_Phalanx.STL
- link Middle_MCP_Pitch: geometry collision mesh filename=meshes/Middle_MCP_Pitch.STL; visual mesh filename=meshes/Middle_MCP_Pitch.STL
- link Middle_MCP_Yaw: geometry collision mesh filename=meshes/collmesh_PIP.STL; visual mesh filename=meshes/Middle_MCP_Yaw.STL
- link Middle_Middle_Phalanx: geometry collision mesh filename=meshes/collmesh_MIP.STL; visual mesh filename=meshes/Middle_Middle_Phalanx.STL
- link Pinky_Distal_Phalanx: geometry collision mesh filename=meshes/collmesh_DIP.STL; visual mesh filename=meshes/Pinky_Distal_Phalanx.STL
- link Pinky_MCP_Pitch: geometry collision mesh filename=meshes/Pinky_MCP_Pitch.STL; visual mesh filename=meshes/Pinky_MCP_Pitch.STL
- link Pinky_MCP_Yaw: geometry collision mesh filename=meshes/collmesh_PIP.STL; visual mesh filename=meshes/Pinky_MCP_Yaw.STL
- link Pinky_Middle_Phalanx: geometry collision mesh filename=meshes/collmesh_MIP.STL; visual mesh filename=meshes/Pinky_Middle_Phalanx.STL
- link Ring_Distal_Phalanx: geometry collision mesh filename=meshes/collmesh_DIP.STL; visual mesh filename=meshes/Ring_Distal_Phalanx.STL
- link Ring_MCP_Pitch: geometry collision mesh filename=meshes/Ring_MCP_Pitch.STL; visual mesh filename=meshes/Ring_MCP_Pitch.STL
- link Ring_MCP_Yaw: geometry collision mesh filename=meshes/collmesh_PIP.STL; visual mesh filename=meshes/Ring_MCP_Yaw.STL
- link Ring_Middle_Phalanx: geometry collision mesh filename=meshes/collmesh_MIP.STL; visual mesh filename=meshes/Ring_Middle_Phalanx.STL
- link Thumb_Distal_Phalanx: geometry collision mesh filename=meshes/collmesh_DIP.STL; visual mesh filename=meshes/Thumb_Distal_Phalanx.STL
- link Thumb_MCP_Pitch: geometry collision mesh filename=meshes/Thumb_MCP_Pitch.STL; visual mesh filename=meshes/Thumb_MCP_Pitch.STL
- link Thumb_MCP_Yaw: geometry collision mesh filename=meshes/collmesh_PIP.STL; visual mesh filename=meshes/Index_MCP_Yaw.STL
- link Thumb_Middle_Phalanx: geometry collision mesh filename=meshes/collmesh_MIP.STL; visual mesh filename=meshes/Index_Middle_Phalanx.STL
- link Thumb_rot: geometry collision mesh filename=meshes/collmesh_thumb_rot.STL; visual mesh filename=meshes/Thumb_rot.STL
- link base_link: geometry collision mesh filename=meshes/collmesh_base_link.STL; visual mesh filename=meshes/base_link.STL
Joints:
- removed joint revolute_Thumb_rot
- added joint revolute_collmesh_thumb_rot: type revolute, parent base_link, child Thumb_rot, origin xyz=0.033806 -0.027174 0.098137 rpy=-0.060476 0.087782 -0.60444, axis 0 0 1, limit lower=-0.35 upper=0.35 effort=0 velocity=0
